File: kit-prisme.kicad_sch (KiCad schematic)
At the start: 95 parts, among them J1 Conn_01x02, J10 Conn_01x03, J11 Conn_01x04, J12 Conn_01x04, J13 Conn_01x04, J14 Conn_01x04, J15 Conn_01x04, J16 Conn_01x04, J17 Conn_01x04, J18 Conn_01x04, J19 Conn_01x04, J2 Conn_01x16, J20 Conn_01x04, J21 Conn_01x04, J22 Conn_01x04, J23 Conn_01x04, J24 Conn_01x04, J25 Conn_01x04, J26 Conn_01x04, J3 Conn_01x16, J4 Conn_01x16, J5 Conn_01x02, J6 Conn_01x02, J7 Conn_01x04, J8 Conn_01x04, J9 Conn_01x04, Q1 2N7000, Q10 2N7000, Q11 2N7000, Q2 2N7000, Q3 2N7000, Q4 2N7000, Q5 2N7000, Q6 2N7000, Q7 2N7000, Q8 2N7000, Q9 2N7000

Commit message: assembling test version, added issue / improvment
Parts:
- R10, R11, R12, R13, R14, R15, R8, R9: value R -> 3K3
- R16, R17, R18, R19, R20, R21, R22, R23: value R -> 27R
Connections:
- net GND: now also Q10.1 (S), Q11.1 (S), Q4.1 (S), Q5.1 (S), Q6.1 (S), Q7.1 (S), Q8.1 (S), Q9.1 (S); no longer Q10.3 (D), Q11.3 (D), Q4.3 (D), Q5.3 (D), Q6.3 (D), Q7.3 (D), Q8.3 (D), Q9.3 (D)
- net at U21.1: now also Q11.3 (D); no longer Q11.1 (S)
- net at U20.1: now also Q10.3 (D); no longer Q10.1 (S)
- net at U18.1: now also Q8.3 (D); no longer Q8.1 (S)
- net at U14.1: now also Q4.3 (D); no longer Q4.1 (S)
- net at U15.1: now also Q5.3 (D); no longer Q5.1 (S)
- net at U19.1: now also Q9.3 (D); no longer Q9.1 (S)
- net at U16.1: now also Q6.3 (D); no longer Q6.1 (S)
- net at U17.1: now also Q7.3 (D); no longer Q7.1 (S)
Other:
- note added: "TO CHECK / FIX -> mosfet orientation -> Mosfet pinout -> spacing J1 -> motor driver module footprint -> width ITR9099 for compatibility -> Vcut for breakoff + solder joint -> Silk note : pin for DC Boost + trimming 5V -> CH340C driver windows -> Dumb proof the battery reverse system, also for lolin... -> move layout of U22 and U13 mux for soldering with encoder -> H-bridge, use red version. Not b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"
- moved on the sheet: Q10, Q11, Q4, Q5, Q6, Q7, Q8, Q9
Changed lines of the file:
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@@
 		)
 	)
+	(text "TO CHECK / FIX\n-> mosfet orientation\n-> Mosfet pinout\n-> spacing J1 \n-> motor driver module footprint\n-> width ITR9099 for compatibility\n-> Vcut for breakoff + solder joint\n-> Silk note : pin for DC Boost + trimming 5V\n-> CH340C driver windows\n-> Dumb proof the battery reverse system, also for lolin...\n-> move layout of U22 and U13 mux for soldering with encoder\n-> H-bridge, use red version. Not black...\n-> Investigate Battery Issue... (lolin has no safety feature...)\n-> ESP32 C3 ? S2 ?\n-> https://de.aliexpress.com/item/1005006823382633.html (charger)\n-> https://de.aliexpress.com/item/1005005374060805.html (1S BMS)"
+		(exclude_from_sim no)
+		(at -5.08 -131.572 0)
+		(effects
+			(font
+				(size 7.62 7.62)
+			)
+			(justify left)
+		)
+	)
 	(text "this is why you have a solder jumper to wire you own supply as needed"
 		(exclude_from_sim no)
@@
 			)
 		)
-		(property "Value" "R"
+		(property "Value" "27R"
 			(at 371.348 90.678 90)
 			(effects
@@
 	(symbol
 		(lib_id "Transistor_FET:2N7000")
-		(at 367.03 245.11 270)
+		(at 367.03 245.11 90)
+		(mirror x)
 		(unit 1)
 		(exclude_from_sim no)
@@
 		(dnp no)
 		(property "Reference" "Q11"
-			(at 361.442 243.078 90)
+			(at 372.618 243.078 90)
 			(effects
 				(font
@@
 		)
 		(property "Value" "2N7000"
-			(at 363.22 250.698 90)
+			(at 370.84 250.698 90)
 			(effects
 				(font
@@
 		)
 		(property "Footprint" "Package_TO_SOT_THT:TO-92_Inline"
-			(at 365.125 250.19 0)
+			(at 368.935 250.19 0)
 			(effects
 				(font
@@
 		)
 		(property "Datasheet" "https://www.vishay.com/docs/70226/70226.pdf"
-			(at 363.22 250.19 0)
+			(at 370.84 250.19 0)
 			(effects
 				(font
@@
 			)
 		)
-		(property "Value" "R"
+		(property "Value" "3K3"
 			(at 317.5 131.318 90)
 			(effects
@@
 	(symbol
 		(lib_id "Transistor_FET:2N7000")
-		(at 367.03 184.15 270)
+		(at 367.03 184.15 90)
+		(mirror x)
 		(unit 1)
 		(exclude_from_sim no)
@@
 		(dnp no)
 		(property "Reference" "Q8"
-			(at 361.442 182.118 90)
+			(at 372.618 182.118 90)
 			(effects
 				(font
@@
 		)
 		(property "Value" "2N7000"
-			(at 363.22 189.738 90)
+			(at 370.84 189.738 90)
 			(effects
 				(font
@@
 		)
 		(property "Footprint" "Package_TO_SOT_THT:TO-92_Inline"
-			(at 365.125 189.23 0)
+			(at 368.935 189.23 0)
 			(effects
 				(font
@@
 		)
 		(property "Datasheet" "https://www.vishay.com/docs/70226/70226.pdf"
-			(at 363.22 189.23 0)
+			(at 370.84 189.23 0)
 			(effects
 				(font
@@
 			)
 		)
-		(property "Value" "R"
+		(property "Value" "3K3"
 			(at 317.5 151.638 90)
 			(effects
@@
 	(symbol
 		(lib_id "Transistor_FET:2N7000")
-		(at 367.03 123.19 270)
+		(at 367.03 123.19 90)
+		(mirror x)
 		(unit 1)
 		(exclude_from_sim no)
@@
 		(dnp no)
 		(property "Reference" "Q5"
-			(at 361.442 121.158 90)
+			(at 372.618 121.158 90)
 			(effects
 				(font
@@
 		)
 		(property "Value" "2N7000"
-			(at 362.966 128.778 90)
+			(at 371.094 128.778 90)
 			(effects
 				(font
@@
 		)
 		(property "Footprint" "Package_TO_SOT_THT:TO-92_Inline"
-			(at 365.125 128.27 0)
+			(at 368.935 128.27 0)
 			(effects
 				(font
@@
 		)
 		(property "Datasheet" "https://www.vishay.com/docs/70226/70226.pdf"
-			(at 363.22 128.27 0)
+			(at 370.84 128.27 0)
 			(effects
 				(font
@@
 			)
 		)
-		(property "Value" "R"
+		(property "Value" "27R"
 			(at 371.348 131.318 90)
 			(effects
@@
 			)
 		)
-		(property "Value" "R"
+		(property "Value" "27R"
 			(at 371.348 110.998 90)
 			(effects
@@
 			)
 		)
-		(property "Value" "R"
+		(property "Value" "27R"
 			(at 371.348 232.918 90)
 			(effects
@@
 	(symbol
 		(lib_id "Transistor_FET:2N7000")
-		(at 367.03 224.79 270)
+		(at 367.03 224.79 90)
+		(mirror x)
 		(unit 1)
 		(exclude_from_sim no)
@@
 		(dnp no)
 		(property "Reference" "Q10"
-			(at 361.442 222.758 90)
+			(at 372.618 222.758 90)
 			(effects
 				(font
@@
 		)
 		(property "Value" "2N7000"
-			(at 362.712 230.378 90)
+			(at 371.348 230.378 90)
 			(effects
 				(font
@@
 		)
 		(property "Footprint" "Package_TO_SOT_THT:TO-92_Inline"
-			(at 365.125 229.87 0)
+			(at 368.935 229.87 0)
 			(effects
 				(font
@@
 		)
 		(property "Datasheet" "https://www.vishay.com/docs/70226/70226.pdf"
-			(at 363.22 229.87 0)
+			(at 370.84 229.87 0)
 			(effects
 				(font
@@
 	(symbol
 		(lib_id "Transistor_FET:2N7000")
-		(at 367.03 204.47 270)
+		(at 367.03 204.47 90)
+		(mirror x)
 		(unit 1)
 		(exclude_from_sim no)
@@
 		(dnp no)
 		(property "Reference" "Q9"
-			(at 361.442 202.438 90)
+			(at 372.618 202.438 90)
 			(effects
 				(font
@@
 		)
 		(property "Value" "2N7000"
-			(at 362.966 210.058 90)
+			(at 371.094 210.058 90)
 			(effects
 				(font
@@
 		)
 		(property "Footprint" "Package_TO_SOT_THT:TO-92_Inline"
-			(at 365.125 209.55 0)
+			(at 368.935 209.55 0)
 			(effects
 				(font
@@
 		)
 		(property "Datasheet" "https://www.vishay.com/docs/70226/70226.pdf"
-			(at 363.22 209.55 0)
+			(at 370.84 209.55 0)
 			(effects
 				(font
@@
 			)
 		)
-		(property "Value" "R"
+		(property "Value" "3K3"
 			(at 317.5 192.278 90)
 			(effects
@@
 			)
 		)
-		(property "Value" "R"
+		(property "Value" "27R"
 			(at 371.348 212.598 90)
 			(effects
@@
 			)
 		)
-		(property "Value" "R"
+		(property "Value" "3K3"
 			(at 317.5 232.918 90)
 			(effects
@@
 			)
 		)
-		(property "Value" "R"
+		(property "Value" "27R"
 			(at 371.348 151.638 90)
 			(effects
@@
 			)
 		)
-		(property "Value" "R"
+		(property "Value" "27R"
 			(at 371.348 171.958 90)
 			(effects
@@
 			)
 		)
-		(property "Value" "R"
+		(property "Value" "3K3"
 			(at 317.5 90.678 90)
 			(effects
@@
 	(symbol
 		(lib_id "Transistor_FET:2N7000")
-		(at 367.03 143.51 270)
+		(at 367.03 143.51 90)
+		(mirror x)
 		(unit 1)
 		(exclude_from_sim no)
@@
 		(dnp no)
 		(property "Reference" "Q6"
-			(at 361.442 141.478 90)
+			(at 372.618 141.478 90)
 			(effects
 				(font
@@
 		)
 		(property "Value" "2N7000"
-			(at 363.728 149.098 90)
+			(at 370.332 149.098 90)
 			(effects
 				(font
@@
 		)
 		(property "Footprint" "Package_TO_SOT_THT:TO-92_Inline"
-			(at 365.125 148.59 0)
+			(at 368.935 148.59 0)
 			(effects
 				(font
@@
 		)
 		(property "Datasheet" "https://www.vishay.com/docs/70226/70226.pdf"
-			(at 363.22 148.59 0)
+			(at 370.84 148.59 0)
 			(effects
 				(font
@@
 	(symbol
 		(lib_id "Transistor_FET:2N7000")
-		(at 367.03 102.87 270)
+		(at 367.03 102.87 90)
+		(mirror x)
 		(unit 1)
 		(exclude_from_sim no)
@@
 		(dnp no)
 		(property "Reference" "Q4"
-			(at 361.442 100.838 90)
+			(at 372.618 100.838 90)
 			(effects
 				(font
@@
 		)
 		(property "Value" "2N7000"
-			(at 362.712 108.458 90)
+			(at 371.348 108.458 90)
 			(effects
 				(font
@@
 		)
 		(property "Footprint" "Package_TO_SOT_THT:TO-92_Inline"
-			(at 365.125 107.95 0)
+			(at 368.935 107.95 0)
 			(effects
 				(font
@@
 		)
 		(property "Datasheet" "https://www.vishay.com/docs/70226/70226.pdf"
-			(at 363.22 107.95 0)
+			(at 370.84 107.95 0)
 			(effects
 				(font
@@
 			)
 		)
-		(property "Value" "R"
+		(property "Value" "3K3"
 			(at 317.5 110.998 90)
 			(effects
@@
 			)
 		)
-		(property "Value" "R"
+		(property "Value" "3K3"
 			(at 317.5 171.958 90)
 			(effects
@@
 			)
 		)
-		(property "Value" "R"
+		(property "Value" "3K3"
 			(at 317.5 212.598 90)
 			(effects
@@
 			)
 		)
-		(property "Value" "R"
+		(property "Value" "27R"
 			(at 371.348 192.278 90)
 			(effects
@@
 	(symbol
 		(lib_id "Transistor_FET:2N7000")
-		(at 367.03 163.83 270)
+		(at 367.03 163.83 90)
+		(mirror x)
 		(unit 1)
 		(exclude_from_sim no)
@@
 		(dnp no)
 		(property "Reference" "Q7"
-			(at 361.442 161.798 90)
+			(at 372.618 161.798 90)
 			(effects
 				(font
@@
 		)
 		(property "Value" "2N7000"
-			(at 362.712 169.418 90)
+			(at 371.348 169.418 90)
 			(effects
 				(font
@@
 		)
 		(property "Footprint" "Package_TO_SOT_THT:TO-92_Inline"
-			(at 365.125 168.91 0)
+			(at 368.935 168.91 0)
 			(effects
 				(font
@@
 		)
 		(property "Datasheet" "https://www.vishay.com/docs/70226/70226.pdf"
-			(at 363.22 168.91 0)
+			(at 370.84 168.91 0)
 			(effects
 				(font
